File: PCB/pcb.kicad_sch (KiCad schematic)
At the start: 201 parts, among them J1 USB_C_Receptacle_USB2.0_16P, SW1 Tab, SW10 Left_Ctrl, SW11 Left_Win, SW12 Left_Alt, SW13 Fn, SW14 Esc, SW15 1, SW16 2, SW17 3, SW18 4, SW19 5, SW2 Caps_Lock, SW20 6, SW21 7, SW22 8, SW23 9, SW24 0, SW25 -, SW26 =, SW27 Q, SW28 W, SW29 E, SW3 Left_Shift, SW30 R, SW31 T, SW32 Y, SW33 U, SW34 I, SW35 O, SW36 P, SW37 [, SW38 ], SW39 \, SW4 Backspace, SW40 A, SW41 S, SW42 D, SW43 F, SW44 G, SW45 H, SW46 J, SW47 K, SW48 L, SW49 ;, SW5 Enter, SW50 ', SW51 Z, SW52 X, SW53 C, SW54 V, SW55 B, SW56 N, SW57 M, SW58 ,, SW59 ., SW6 Right_Shift, SW60 /, SW61 MENU, SW62 Boot, SW63 Reset, SW7 Spacebar, SW8 Right_Ctrl, SW9 Right_Alt, U1 STM32F072C8Tx, U2 ER_OLEDM0.91_1x-I2C, U3 AMS1117-3.3, U4 USBLC6-2SC6

Commit message: Introducing... Tachi Ninja V2
Parts:
- SW1: value Tab -> ESC; footprint Button_Switch_Keyboard:SW_Cherry_MX_1.50u_PCB -> Switch_Keyboard_Hotswap_Kailh:SW_Hotswap_Kailh_MX_1.00u
- SW10: value Left_Ctrl -> 9; footprint Button_Switch_Keyboard:SW_Cherry_MX_1.25u_PCB -> Switch_Keyboard_Hotswap_Kailh:SW_Hotswap_Kailh_MX_1.00u
- SW11: value Left_Win -> 0; footprint Button_Switch_Keyboard:SW_Cherry_MX_1.25u_PCB -> Switch_Keyboard_Hotswap_Kailh:SW_Hotswap_Kailh_MX_1.00u
- SW12: value Left_Alt -> -; footprint Button_Switch_Keyboard:SW_Cherry_MX_1.25u_PCB -> Switch_Keyboard_Hotswap_Kailh:SW_Hotswap_Kailh_MX_1.00u
- SW13: value Fn -> =; footprint Button_Switch_Keyboard:SW_Cherry_MX_1.25u_PCB -> Switch_Keyboard_Hotswap_Kailh:SW_Hotswap_Kailh_MX_1.00u
- SW14: value Esc -> BACKSPACE; footprint Button_Switch_Keyboard:SW_Cherry_MX_1.00u_PCB -> Switch_Keyboard_Hotswap_Kailh:SW_Hotswap_Kailh_MX_2.00u
- SW15: value 1 -> TAB; footprint Button_Switch_Keyboard:SW_Cherry_MX_1.00u_PCB -> Switch_Keyboard_Hotswap_Kailh:SW_Hotswap_Kailh_MX_1.50u
- SW16: value 2 -> Q; footprint Button_Switch_Keyboard:SW_Cherry_MX_1.00u_PCB -> Switch_Keyboard_Hotswap_Kailh:SW_Hotswap_Kailh_MX_1.00u
- SW17: value 3 -> W; footprint Button_Switch_Keyboard:SW_Cherry_MX_1.00u_PCB -> Switch_Keyboard_Hotswap_Kailh:SW_Hotswap_Kailh_MX_1.00u
- SW18: value 4 -> E; footprint Button_Switch_Keyboard:SW_Cherry_MX_1.00u_PCB -> Switch_Keyboard_Hotswap_Kailh:SW_Hotswap_Kailh_MX_1.00u
- SW19: value 5 -> R; footprint Button_Switch_Keyboard:SW_Cherry_MX_1.00u_PCB -> Switch_Keyboard_Hotswap_Kailh:SW_Hotswap_Kailh_MX_1.00u
- SW2: value Caps_Lock -> 1; footprint Button_Switch_Keyboard:SW_Cherry_MX_1.75u_PCB -> Switch_Keyboard_Hotswap_Kailh:SW_Hotswap_Kailh_MX_1.00u
- SW20: value 6 -> T; footprint Button_Switch_Keyboard:SW_Cherry_MX_1.00u_PCB -> Switch_Keyboard_Hotswap_Kailh:SW_Hotswap_Kailh_MX_1.00u
- SW21: value 7 -> Y; footprint Button_Switch_Keyboard:SW_Cherry_MX_1.00u_PCB -> Switch_Keyboard_Hotswap_Kailh:SW_Hotswap_Kailh_MX_1.00u
- SW22: value 8 -> U; footprint Button_Switch_Keyboard:SW_Cherry_MX_1.00u_PCB -> Switch_Keyboard_Hotswap_Kailh:SW_Hotswap_Kailh_MX_1.00u
- SW23: value 9 -> I; footprint Button_Switch_Keyboard:SW_Cherry_MX_1.00u_PCB -> Switch_Keyboard_Hotswap_Kailh:SW_Hotswap_Kailh_MX_1.00u
- SW24: value 0 -> O; footprint Button_Switch_Keyboard:SW_Cherry_MX_1.00u_PCB -> Switch_Keyboard_Hotswap_Kailh:SW_Hotswap_Kailh_MX_1.00u
- SW25: value - -> P; footprint Button_Switch_Keyboard:SW_Cherry_MX_1.00u_PCB -> Switch_Keyboard_Hotswap_Kailh:SW_Hotswap_Kailh_MX_1.00u
- SW26: value = -> [; footprint Button_Switch_Keyboard:SW_Cherry_MX_1.00u_PCB -> Switch_Keyboard_Hotswap_Kailh:SW_Hotswap_Kailh_MX_1.00u
- SW27: value Q -> ]; footprint Button_Switch_Keyboard:SW_Cherry_MX_1.00u_PCB -> Switch_Keyboard_Hotswap_Kailh:SW_Hotswap_Kailh_MX_1.00u
- SW28: value W -> \; footprint Button_Switch_Keyboard:SW_Cherry_MX_1.00u_PCB -> Switch_Keyboard_Hotswap_Kailh:SW_Hotswap_Kailh_MX_1.50u
- SW29: value E -> CAPSLOCK; footprint Button_Switch_Keyboard:SW_Cherry_MX_1.00u_PCB -> Switch_Keyboard_Hotswap_Kailh:SW_Hotswap_Kailh_MX_1.75u
- SW3: value Left_Shift -> 2; footprint Button_Switch_Keyboard:SW_Cherry_MX_2.25u_PCB -> Switch_Keyboard_Hotswap_Kailh:SW_Hotswap_Kailh_MX_1.00u
- SW30: value R -> A; footprint Button_Switch_Keyboard:SW_Cherry_MX_1.00u_PCB -> Switch_Keyboard_Hotswap_Kailh:SW_Hotswap_Kailh_MX_1.00u
- SW31: value T -> S; footprint Button_Switch_Keyboard:SW_Cherry_MX_1.00u_PCB -> Switch_Keyboard_Hotswap_Kailh:SW_Hotswap_Kailh_MX_1.00u
- SW32: value Y -> D; footprint Button_Switch_Keyboard:SW_Cherry_MX_1.00u_PCB -> Switch_Keyboard_Hotswap_Kailh:SW_Hotswap_Kailh_MX_1.00u
- SW33: value U -> F; footprint Button_Switch_Keyboard:SW_Cherry_MX_1.00u_PCB -> Switch_Keyboard_Hotswap_Kailh:SW_Hotswap_Kailh_MX_1.00u
- SW34: value I -> G; footprint Button_Switch_Keyboard:SW_Cherry_MX_1.00u_PCB -> Switch_Keyboard_Hotswap_Kailh:SW_Hotswap_Kailh_MX_1.00u
- SW35: value O -> H; footprint Button_Switch_Keyboard:SW_Cherry_MX_1.00u_PCB -> Switch_Keyboard_Hotswap_Kailh:SW_Hotswap_Kailh_MX_1.00u
- SW36: value P -> J; footprint Button_Switch_Keyboard:SW_Cherry_MX_1.00u_PCB -> Switch_Keyboard_Hotswap_Kailh:SW_Hotswap_Kailh_MX_1.00u
- SW37: value [ -> K; footprint Button_Switch_Keyboard:SW_Cherry_MX_1.00u_PCB -> Switch_Keyboard_Hotswap_Kailh:SW_Hotswap_Kailh_MX_1.00u
- SW38: value ] -> L; footprint Button_Switch_Keyboard:SW_Cherry_MX_1.00u_PCB -> Switch_Keyboard_Hotswap_Kailh:SW_Hotswap_Kailh_MX_1.00u
- SW39: value \ -> ;; footprint Button_Switch_Keyboard:SW_Cherry_MX_1.50u_PCB -> Switch_Keyboard_Hotswap_Kailh:SW_Hotswap_Kailh_MX_1.00u
- SW4: value Backspace -> 3; footprint Button_Switch_Keyboard:SW_Cherry_MX_2.00u_PCB -> Switch_Keyboard_Hotswap_Kailh:SW_Hotswap_Kailh_MX_1.00u
- SW40: value A -> '; footprint Button_Switch_Keyboard:SW_Cherry_MX_1.00u_PCB -> Switch_Keyboard_Hotswap_Kailh:SW_Hotswap_Kailh_MX_1.00u
- SW41: value S -> ENTER; footprint Button_Switch_Keyboard:SW_Cherry_MX_1.00u_PCB -> Switch_Keyboard_Hotswap_Kailh:SW_Hotswap_Kailh_MX_2.25u
- SW42: value D -> LEFTSHIFT; footprint Button_Switch_Keyboard:SW_Cherry_MX_1.00u_PCB -> Switch_Keyboard_Hotswap_Kailh:SW_Hotswap_Kailh_MX_2.25u
- SW43: value F -> Z; footprint Button_Switch_Keyboard:SW_Cherry_MX_1.00u_PCB -> Switch_Keyboard_Hotswap_Kailh:SW_Hotswap_Kailh_MX_1.00u
- SW44: value G -> X; footprint Button_Switch_Keyboard:SW_Cherry_MX_1.00u_PCB -> Switch_Keyboard_Hotswap_Kailh:SW_Hotswap_Kailh_MX_1.00u
- SW45: value H -> C; footprint Button_Switch_Keyboard:SW_Cherry_MX_1.00u_PCB -> Switch_Keyboard_Hotswap_Kailh:SW_Hotswap_Kailh_MX_1.00u
- SW46: value J -> V; footprint Button_Switch_Keyboard:SW_Cherry_MX_1.00u_PCB -> Switch_Keyboard_Hotswap_Kailh:SW_Hotswap_Kailh_MX_1.00u
- SW47: value K -> B; footprint Button_Switch_Keyboard:SW_Cherry_MX_1.00u_PCB -> Switch_Keyboard_Hotswap_Kailh:SW_Hotswap_Kailh_MX_1.00u
- SW48: value L -> N; footprint Button_Switch_Keyboard:SW_Cherry_MX_1.00u_PCB -> Switch_Keyboard_Hotswap_Kailh:SW_Hotswap_Kailh_MX_1.00u
- SW49: value ; -> M; footprint Button_Switch_Keyboard:SW_Cherry_MX_1.00u_PCB -> Switch_Keyboard_Hotswap_Kailh:SW_Hotswap_Kailh_MX_1.00u
- SW5: value Enter -> 4; footprint Button_Switch_Keyboard:SW_Cherry_MX_2.25u_PCB -> Switch_Keyboard_Hotswap_Kailh:SW_Hotswap_Kailh_MX_1.00u
- SW50: value ' -> ,; footprint Button_Switch_Keyboard:SW_Cherry_MX_1.00u_PCB -> Switch_Keyboard_Hotswap_Kailh:SW_Hotswap_Kailh_MX_1.00u
- SW51: value Z -> .; footprint Button_Switch_Keyboard:SW_Cherry_MX_1.00u_PCB -> Switch_Keyboard_Hotswap_Kailh:SW_Hotswap_Kailh_MX_1.00u
- SW52: value X -> /; footprint Button_Switch_Keyboard:SW_Cherry_MX_1.00u_PCB -> Switch_Keyboard_Hotswap_Kailh:SW_Hotswap_Kailh_MX_1.00u
- SW53: value C -> RIGHTSHIFT; footprint Button_Switch_Keyboard:SW_Cherry_MX_1.00u_PCB -> Switch_Keyboard_Hotswap_Kailh:SW_Hotswap_Kailh_MX_2.75u
- SW54: value V -> LEFTCTRL; footprint Button_Switch_Keyboard:SW_Cherry_MX_1.00u_PCB -> Switch_Keyboard_Hotswap_Kailh:SW_Hotswap_Kailh_MX_1.25u
- SW55: value B -> LEFTWIN; footprint Button_Switch_Keyboard:SW_Cherry_MX_1.00u_PCB -> Switch_Keyboard_Hotswap_Kailh:SW_Hotswap_Kailh_MX_1.25u
- SW56: value N -> LEFTALT; footprint Button_Switch_Keyboard:SW_Cherry_MX_1.00u_PCB -> Switch_Keyboard_Hotswap_Kailh:SW_Hotswap_Kailh_MX_1.25u
- SW57: value M -> SPACE; footprint Button_Switch_Keyboard:SW_Cherry_MX_1.00u_PCB -> Switch_Keyboard_Hotswap_Kailh:SW_Hotswap_Kailh_MX_6.25u
- SW58: value , -> RIGHTALT; footprint Button_Switch_Keyboard:SW_Cherry_MX_1.00u_PCB -> Switch_Keyboard_Hotswap_Kailh:SW_Hotswap_Kailh_MX_1.25u
- SW59: value . -> FN; footprint Button_Switch_Keyboard:SW_Cherry_MX_1.00u_PCB -> Switch_Keyboard_Hotswap_Kailh:SW_Hotswap_Kailh_MX_1.25u
- SW6: value Right_Shift -> 5; footprint Button_Switch_Keyboard:SW_Cherry_MX_2.75u_PCB -> Switch_Keyboard_Hotswap_Kailh:SW_Hotswap_Kailh_MX_1.00u
- SW60: value / -> MENU; footprint Button_Switch_Keyboard:SW_Cherry_MX_1.00u_PCB -> Switch_Keyboard_Hotswap_Kailh:SW_Hotswap_Kailh_MX_1.25u
- SW61: value MENU -> RIGHTCTRL; footprint Button_Switch_Keyboard:SW_Cherry_MX_1.25u_PCB -> Switch_Keyboard_Hotswap_Kailh:SW_Hotswap_Kailh_MX_1.25u
- SW7: value Spacebar -> 6; footprint Button_Switch_Keyboard:SW_Cherry_MX_6.25u_PCB -> Switch_Keyboard_Hotswap_Kailh:SW_Hotswap_Kailh_MX_1.00u
- SW8: value Right_Ctrl -> 7; footprint Button_Switch_Keyboard:SW_Cherry_MX_1.25u_PCB -> Switch_Keyboard_Hotswap_Kailh:SW_Hotswap_Kailh_MX_1.00u
- SW9: value Right_Alt -> 8; footprint Button_Switch_Keyboard:SW_Cherry_MX_1.25u_PCB -> Switch_Keyboard_Hotswap_Kailh:SW_Hotswap_Kailh_MX_1.00u
Connections:
- net COL12: no longer D156.2 (A)
- net COL13: now also D156.2 (A)
- net ROW0: now also SW1.2, SW10.2, SW11.2, SW12.2, SW13.2, SW2.2, SW3.2, SW5.2, SW6.2, SW7.2, SW8.2, SW9.2; no longer SW15.2, SW16.2, SW17.2, SW18.2, SW19.2, SW20.2, SW21.2, SW22.2, SW23.2, SW24.2, SW25.2, SW26.2
- net ROW1: now also SW15.2, SW16.2, SW17.2, SW18.2, SW19.2, SW20.2, SW21.2, SW22.2, SW23.2, SW24.2, SW25.2, SW26.2; no longer SW1.2, SW29.2, SW30.2, SW31.2, SW32.2, SW33.2, SW34.2, SW35.2, SW36.2, SW37.2, SW38.2, SW39.2
- net ROW2: now also SW29.2, SW30.2, SW31.2, SW32.2, SW33.2, SW34.2, SW35.2, SW36.2, SW37.2, SW38.2, SW39.2; no longer SW2.2, SW42.2, SW43.2, SW44.2, SW45.2, SW46.2, SW47.2, SW48.2, SW49.2, SW5.2, SW50.2
- net ROW3: now also SW42.2, SW43.2, SW44.2, SW45.2, SW46.2, SW47.2, SW48.2, SW49.2, SW50.2; no longer SW3.2, SW54.2, SW55.2, SW56.2, SW57.2, SW58.2, SW59.2, SW6.2, SW60.2
- net ROW4: now also SW54.2, SW55.2, SW56.2, SW57.2, SW58.2, SW59.2, SW60.2; no longer SW10.2, SW11.2, SW12.2, SW13.2, SW7.2, SW8.2, SW9.2
- net at D103.1 (K): now also SW6.1; no longer SW19.1
- net at D161.1 (K): now also SW14.1; no longer SW4.1
- net at SW53.1: now also D150.1 (K); no longer D90.1 (K)
- net at D165.1 (K): now also SW61.1; no longer SW8.1
- net at SW49.1: now also D122.1 (K); no longer D142.1 (K)
- net at D149.1 (K): now also SW40.1; no longer SW50.1
- net at D89.1 (K): now also SW32.1; no longer SW42.1
- net at D88.1 (K): now also SW18.1; no longer SW29.1
- net at D105.1 (K): now also SW34.1; no longer SW44.1
- net at SW36.1: now also D121.1 (K); no longer D141.1 (K)
- net at D151.1 (K): now also SW59.1; no longer SW61.1
- net at D119.1 (K): now also SW8.1; no longer SW21.1
- net at D140.1 (K): now also SW11.1; no longer SW24.1
- net at SW10.1: now also D133.1 (K); no longer D67.1 (K)
- net at D74.1 (K): now also SW43.1; no longer SW51.1
- net at SW46.1: now also D98.1 (K); no longer D121.1 (K)
- net at D127.1 (K): now also SW23.1; no longer SW34.1
- net at D104.1 (K): now also SW20.1; no longer SW31.1
- net at SW15.1: now also D64.1 (K); no longer D71.1 (K)
- net at D148.1 (K): now also SW26.1; no longer SW37.1
- net at SW45.1: now also D90.1 (K); no longer D113.1 (K)
- net at D156.1 (K): now also SW41.1; no longer SW5.1
- net at SW1.1: now also D63.1 (K); no longer D64.1 (K)
- net at SW7.1: now also D111.1 (K); no longer D115.1 (K)
- net at SW38.1: now also D135.1 (K); no longer D155.1 (K)
- net at SW33.1: now also D97.1 (K); no longer D120.1 (K)
- net at D75.1 (K): now also SW55.1; no longer SW11.1
- net at D95.1 (K): now also SW5.1; no longer SW18.1
- net at D144.1 (K): now also SW58.1; no longer SW9.1
- net at SW30.1: now also D73.1 (K); no longer D96.1 (K)
- net at D154.1 (K): now also SW13.1; no longer SW26.1
- net at SW35.1: now also D113.1 (K); no longer D134.1 (K)
- net at D129.1 (K): now also SW50.1; no longer SW58.1
- net at D106.1 (K): now also SW47.1; no longer SW55.1
- net at D66.1 (K): now also SW42.1; no longer SW3.1
- net at SW39.1: now also D142.1 (K); no longer D162.1 (K)
- net at SW56.1: now also D83.1 (K); no longer D114.1 (K)
- net at SW22.1: now also D120.1 (K); no longer D126.1 (K)
- net at SW57.1: now also D115.1 (K); no longer D122.1 (K)
- net at SW28.1: now also D162.1 (K); no longer D80.1 (K)
- net at D72.1 (K): now also SW16.1; no longer SW27.1
- net at SW48.1: now also D114.1 (K); no longer D135.1 (K)
- net at SW2.1: now also D71.1 (K); no longer D65.1 (K)
- net at D143.1 (K): now also SW52.1; no longer SW60.1
- net at D112.1 (K): now also SW21.1; no longer SW32.1
- net at D87.1 (K): now also SW4.1; no longer SW17.1
- net at D79.1 (K): now also SW3.1; no longer SW16.1
- net at D81.1 (K): now also SW31.1; no longer SW41.1
- net at D136.1 (K): now also SW51.1; no longer SW59.1
- net at SW54.1: now also D67.1 (K); no longer D98.1 (K)
- net at D128.1 (K): now also SW37.1; no longer SW47.1
- net at D82.1 (K): now also SW44.1; no longer SW52.1
- net at D158.1 (K): now also SW60.1; no longer SW13.1
- net at SW12.1: now also D147.1 (K); no longer D83.1 (K)
- net at SW25.1: now also D141.1 (K); no longer D147.1 (K)
- new net: D80.1 (K), SW17.1
- new net: D134.1 (K), SW24.1
- new net: D126.1 (K), SW9.1
- new net: D155.1 (K), SW27.1
- new net: D65.1 (K), SW29.1
- new net: D96.1 (K), SW19.1
Other:
- moved on the sheet: D156
