File: PCB/pcb.kicad_pcb (KiCad board)
At the start: 2 copper layers, 305.9 x 124.4 mm, 205 parts, among them J1 USB_C_Receptacle_USB2.0_16P, SW1 Tab, SW10 Left_Ctrl, SW11 Left_Win, SW12 Left_Alt, SW13 Fn, SW14 Esc, SW15 1, SW16 2, SW17 3, SW18 4, SW19 5, SW2 Caps_Lock, SW20 6, SW21 7, SW22 8, SW23 9, SW24 0, SW25 -, SW26 =, SW27 Q, SW28 W, SW29 E, SW3 Left_Shift, SW30 R, SW31 T, SW32 Y, SW33 U, SW34 I, SW35 O, SW36 P, SW37 [, SW38 ], SW39 \, SW4 Backspace, SW40 A, SW41 S, SW42 D, SW43 F, SW44 G, SW45 H, SW46 J, SW47 K, SW48 L, SW49 ;, SW5 Enter, SW50 ', SW51 Z, SW52 X, SW53 C, SW54 V, SW55 B, SW56 N, SW57 M, SW58 ,, SW59 ., SW6 Right_Shift, SW60 /, SW61 MENU, SW7 Spacebar, SW8 Right_Ctrl, SW9 Right_Alt, U1 STM32F072C8Tx, U2 ER_OLEDM0.91_1x-I2C, U3 AMS1117-3.3, U4 USBLC6-2SC6

Commit message: Introducing... Tachi Ninja V2
Parts:
- removed Boot: Boot, Button_Switch_SMD:SW_SPST_B3U-1000P
- removed the REF** at (98.5, 31.0)
- removed the REF** at (395.9, 30.6)
- removed the REF** at (395.0, 145.8)
- removed the REF** at (98.1, 146.8)
- removed Reset: Reset, Button_Switch_SMD:SW_SPST_B3U-1000P
- added REF**: Stabilizer_Cherry_MX_3.00u, Mounting_Keyboard_Stabilizer:Stabilizer_Cherry_MX_3.00u, F.Cu at (316.2, 137.0)
- added REF**: Stabilizer_Cherry_MX_2.00u, Mounting_Keyboard_Stabilizer:Stabilizer_Cherry_MX_2.00u, F.Cu at (73.2, 137.0)
- added REF**: Stabilizer_Cherry_MX_2.00u, Mounting_Keyboard_Stabilizer:Stabilizer_Cherry_MX_2.00u, F.Cu at (324.4, 78.3)
- added REF**: MountingHole_3.2mm_M3, MountingHole:MountingHole_3.2mm_M3, F.Cu at (347.5, 168.0)
- added REF**: MountingHole_3.2mm_M3, MountingHole:MountingHole_3.2mm_M3, F.Cu at (47.5, 167.5)
- added REF**: MountingHole_3.2mm_M3, MountingHole:MountingHole_3.2mm_M3, F.Cu at (47.0, 47.0)
- added REF**: Stabilizer_Cherry_MX_2.00u, Mounting_Keyboard_Stabilizer:Stabilizer_Cherry_MX_2.00u, F.Cu at (321.2, 117.0)
- added REF**: MountingHole_3.2mm_M3, MountingHole:MountingHole_3.2mm_M3, F.Cu at (347.5, 47.0)
- added REF**: Stabilizer_Cherry_MX_6.25u, Mounting_Keyboard_Stabilizer:Stabilizer_Cherry_MX_6.25u, F.Cu at (185.2, 157.0)
- added SW62: Boot, Button_Switch_SMD:SW_SPST_B3U-1000P, F.Cu at (325.7, 54.0)
- added SW63: Reset, Button_Switch_SMD:SW_SPST_B3U-1000P, F.Cu at (330.8, 54.0)
- R1, R2: moved to B.Cu
- SW1: value Tab -> ESC; footprint Button_Switch_Keyboard:SW_Cherry_MX_1.50u_PCB -> Switch_Keyboard_Hotswap_Kailh:SW_Hotswap_Kailh_MX_1.00u
- SW10: value Left_Ctrl -> 9; footprint Button_Switch_Keyboard:SW_Cherry_MX_1.25u_PCB -> Switch_Keyboard_Hotswap_Kailh:SW_Hotswap_Kailh_MX_1.00u
- SW11: value Left_Win -> 0; footprint Button_Switch_Keyboard:SW_Cherry_MX_1.25u_PCB -> Switch_Keyboard_Hotswap_Kailh:SW_Hotswap_Kailh_MX_1.00u
- SW12: value Left_Alt -> -; footprint Button_Switch_Keyboard:SW_Cherry_MX_1.25u_PCB -> Switch_Keyboard_Hotswap_Kailh:SW_Hotswap_Kailh_MX_1.00u
- SW13: value Fn -> =; footprint Button_Switch_Keyboard:SW_Cherry_MX_1.25u_PCB -> Switch_Keyboard_Hotswap_Kailh:SW_Hotswap_Kailh_MX_1.00u
- SW14: value Esc -> BACKSPACE; footprint Button_Switch_Keyboard:SW_Cherry_MX_1.00u_PCB -> Switch_Keyboard_Hotswap_Kailh:SW_Hotswap_Kailh_MX_2.00u
- SW15: value 1 -> TAB; footprint Button_Switch_Keyboard:SW_Cherry_MX_1.00u_PCB -> Switch_Keyboard_Hotswap_Kailh:SW_Hotswap_Kailh_MX_1.50u
- SW16: value 2 -> Q; footprint Button_Switch_Keyboard:SW_Cherry_MX_1.00u_PCB -> Switch_Keyboard_Hotswap_Kailh:SW_Hotswap_Kailh_MX_1.00u
- SW17: value 3 -> W; footprint Button_Switch_Keyboard:SW_Cherry_MX_1.00u_PCB -> Switch_Keyboard_Hotswap_Kailh:SW_Hotswap_Kailh_MX_1.00u
- SW18: value 4 -> E; footprint Button_Switch_Keyboard:SW_Cherry_MX_1.00u_PCB -> Switch_Keyboard_Hotswap_Kailh:SW_Hotswap_Kailh_MX_1.00u
- SW19: value 5 -> R; footprint Button_Switch_Keyboard:SW_Cherry_MX_1.00u_PCB -> Switch_Keyboard_Hotswap_Kailh:SW_Hotswap_Kailh_MX_1.00u
- SW2: value Caps_Lock -> 1; footprint Button_Switch_Keyboard:SW_Cherry_MX_1.75u_PCB -> Switch_Keyboard_Hotswap_Kailh:SW_Hotswap_Kailh_MX_1.00u
- SW20: value 6 -> T; footprint Button_Switch_Keyboard:SW_Cherry_MX_1.00u_PCB -> Switch_Keyboard_Hotswap_Kailh:SW_Hotswap_Kailh_MX_1.00u
- SW21: value 7 -> Y; footprint Button_Switch_Keyboard:SW_Cherry_MX_1.00u_PCB -> Switch_Keyboard_Hotswap_Kailh:SW_Hotswap_Kailh_MX_1.00u
- SW22: value 8 -> U; footprint Button_Switch_Keyboard:SW_Cherry_MX_1.00u_PCB -> Switch_Keyboard_Hotswap_Kailh:SW_Hotswap_Kailh_MX_1.00u
- SW23: value 9 -> I; footprint Button_Switch_Keyboard:SW_Cherry_MX_1.00u_PCB -> Switch_Keyboard_Hotswap_Kailh:SW_Hotswap_Kailh_MX_1.00u
- SW24: value 0 -> O; footprint Button_Switch_Keyboard:SW_Cherry_MX_1.00u_PCB -> Switch_Keyboard_Hotswap_Kailh:SW_Hotswap_Kailh_MX_1.00u
- SW25: value - -> P; footprint Button_Switch_Keyboard:SW_Cherry_MX_1.00u_PCB -> Switch_Keyboard_Hotswap_Kailh:SW_Hotswap_Kailh_MX_1.00u
- SW26: value = -> [; footprint Button_Switch_Keyboard:SW_Cherry_MX_1.00u_PCB -> Switch_Keyboard_Hotswap_Kailh:SW_Hotswap_Kailh_MX_1.00u
- SW27: value Q -> ]; footprint Button_Switch_Keyboard:SW_Cherry_MX_1.00u_PCB -> Switch_Keyboard_Hotswap_Kailh:SW_Hotswap_Kailh_MX_1.00u
- SW28: value W -> \; footprint Button_Switch_Keyboard:SW_Cherry_MX_1.00u_PCB -> Switch_Keyboard_Hotswap_Kailh:SW_Hotswap_Kailh_MX_1.50u
- SW29: value E -> CAPSLOCK; footprint Button_Switch_Keyboard:SW_Cherry_MX_1.00u_PCB -> Switch_Keyboard_Hotswap_Kailh:SW_Hotswap_Kailh_MX_1.75u
- SW3: value Left_Shift -> 2; footprint Button_Switch_Keyboard:SW_Cherry_MX_2.25u_PCB -> Switch_Keyboard_Hotswap_Kailh:SW_Hotswap_Kailh_MX_1.00u
- SW30: value R -> A; footprint Button_Switch_Keyboard:SW_Cherry_MX_1.00u_PCB -> Switch_Keyboard_Hotswap_Kailh:SW_Hotswap_Kailh_MX_1.00u
- SW31: value T -> S; footprint Button_Switch_Keyboard:SW_Cherry_MX_1.00u_PCB -> Switch_Keyboard_Hotswap_Kailh:SW_Hotswap_Kailh_MX_1.00u
- SW32: value Y -> D; footprint Button_Switch_Keyboard:SW_Cherry_MX_1.00u_PCB -> Switch_Keyboard_Hotswap_Kailh:SW_Hotswap_Kailh_MX_1.00u
- SW33: value U -> F; footprint Button_Switch_Keyboard:SW_Cherry_MX_1.00u_PCB -> Switch_Keyboard_Hotswap_Kailh:SW_Hotswap_Kailh_MX_1.00u
- SW34: value I -> G; footprint Button_Switch_Keyboard:SW_Cherry_MX_1.00u_PCB -> Switch_Keyboard_Hotswap_Kailh:SW_Hotswap_Kailh_MX_1.00u
- SW35: value O -> H; footprint Button_Switch_Keyboard:SW_Cherry_MX_1.00u_PCB -> Switch_Keyboard_Hotswap_Kailh:SW_Hotswap_Kailh_MX_1.00u
- SW36: value P -> J; footprint Button_Switch_Keyboard:SW_Cherry_MX_1.00u_PCB -> Switch_Keyboard_Hotswap_Kailh:SW_Hotswap_Kailh_MX_1.00u
- SW37: value [ -> K; footprint Button_Switch_Keyboard:SW_Cherry_MX_1.00u_PCB -> Switch_Keyboard_Hotswap_Kailh:SW_Hotswap_Kailh_MX_1.00u
- SW38: value ] -> L; footprint Button_Switch_Keyboard:SW_Cherry_MX_1.00u_PCB -> Switch_Keyboard_Hotswap_Kailh:SW_Hotswap_Kailh_MX_1.00u
- SW39: value \ -> ;; footprint Button_Switch_Keyboard:SW_Cherry_MX_1.50u_PCB -> Switch_Keyboard_Hotswap_Kailh:SW_Hotswap_Kailh_MX_1.00u
- SW4: value Backspace -> 3; footprint Button_Switch_Keyboard:SW_Cherry_MX_2.00u_PCB -> Switch_Keyboard_Hotswap_Kailh:SW_Hotswap_Kailh_MX_1.00u
- SW40: value A -> '; footprint Button_Switch_Keyboard:SW_Cherry_MX_1.00u_PCB -> Switch_Keyboard_Hotswap_Kailh:SW_Hotswap_Kailh_MX_1.00u
- SW41: value S -> ENTER; footprint Button_Switch_Keyboard:SW_Cherry_MX_1.00u_PCB -> Switch_Keyboard_Hotswap_Kailh:SW_Hotswap_Kailh_MX_2.25u
- SW42: value D -> LEFTSHIFT; footprint Button_Switch_Keyboard:SW_Cherry_MX_1.00u_PCB -> Switch_Keyboard_Hotswap_Kailh:SW_Hotswap_Kailh_MX_2.25u
- SW43: value F -> Z; footprint Button_Switch_Keyboard:SW_Cherry_MX_1.00u_PCB -> Switch_Keyboard_Hotswap_Kailh:SW_Hotswap_Kailh_MX_1.00u
- SW44: value G -> X; footprint Button_Switch_Keyboard:SW_Cherry_MX_1.00u_PCB -> Switch_Keyboard_Hotswap_Kailh:SW_Hotswap_Kailh_MX_1.00u
- SW45: value H -> C; footprint Button_Switch_Keyboard:SW_Cherry_MX_1.00u_PCB -> Switch_Keyboard_Hotswap_Kailh:SW_Hotswap_Kailh_MX_1.00u
- SW46: value J -> V; footprint Button_Switch_Keyboard:SW_Cherry_MX_1.00u_PCB -> Switch_Keyboard_Hotswap_Kailh:SW_Hotswap_Kailh_MX_1.00u
- SW47: value K -> B; footprint Button_Switch_Keyboard:SW_Cherry_MX_1.00u_PCB -> Switch_Keyboard_Hotswap_Kailh:SW_Hotswap_Kailh_MX_1.00u
- SW48: value L -> N; footprint Button_Switch_Keyboard:SW_Cherry_MX_1.00u_PCB -> Switch_Keyboard_Hotswap_Kailh:SW_Hotswap_Kailh_MX_1.00u
- SW49: value ; -> M; footprint Button_Switch_Keyboard:SW_Cherry_MX_1.00u_PCB -> Switch_Keyboard_Hotswap_Kailh:SW_Hotswap_Kailh_MX_1.00u
- SW5: value Enter -> 4; footprint Button_Switch_Keyboard:SW_Cherry_MX_2.25u_PCB -> Switch_Keyboard_Hotswap_Kailh:SW_Hotswap_Kailh_MX_1.00u
- SW50: value ' -> ,; footprint Button_Switch_Keyboard:SW_Cherry_MX_1.00u_PCB -> Switch_Keyboard_Hotswap_Kailh:SW_Hotswap_Kailh_MX_1.00u
- SW51: value Z -> .; footprint Button_Switch_Keyboard:SW_Cherry_MX_1.00u_PCB -> Switch_Keyboard_Hotswap_Kailh:SW_Hotswap_Kailh_MX_1.00u
- SW52: value X -> /; footprint Button_Switch_Keyboard:SW_Cherry_MX_1.00u_PCB -> Switch_Keyboard_Hotswap_Kailh:SW_Hotswap_Kailh_MX_1.00u
- SW53: value C -> RIGHTSHIFT; footprint Button_Switch_Keyboard:SW_Cherry_MX_1.00u_PCB -> Switch_Keyboard_Hotswap_Kailh:SW_Hotswap_Kailh_MX_2.75u
- SW54: value V -> LEFTCTRL; footprint Button_Switch_Keyboard:SW_Cherry_MX_1.00u_PCB -> Switch_Keyboard_Hotswap_Kailh:SW_Hotswap_Kailh_MX_1.25u
- SW55: value B -> LEFTWIN; footprint Button_Switch_Keyboard:SW_Cherry_MX_1.00u_PCB -> Switch_Keyboard_Hotswap_Kailh:SW_Hotswap_Kailh_MX_1.25u
- SW56: value N -> LEFTALT; footprint Button_Switch_Keyboard:SW_Cherry_MX_1.00u_PCB -> Switch_Keyboard_Hotswap_Kailh:SW_Hotswap_Kailh_MX_1.25u
- SW57: value M -> SPACE; footprint Button_Switch_Keyboard:SW_Cherry_MX_1.00u_PCB -> Switch_Keyboard_Hotswap_Kailh:SW_Hotswap_Kailh_MX_6.25u
- SW58: value , -> RIGHTALT; footprint Button_Switch_Keyboard:SW_Cherry_MX_1.00u_PCB -> Switch_Keyboard_Hotswap_Kailh:SW_Hotswap_Kailh_MX_1.25u
- SW59: value . -> FN; footprint Button_Switch_Keyboard:SW_Cherry_MX_1.00u_PCB -> Switch_Keyboard_Hotswap_Kailh:SW_Hotswap_Kailh_MX_1.25u
- SW6: value Right_Shift -> 5; footprint Button_Switch_Keyboard:SW_Cherry_MX_2.75u_PCB -> Switch_Keyboard_Hotswap_Kailh:SW_Hotswap_Kailh_MX_1.00u
- SW60: value / -> MENU; footprint Button_Switch_Keyboard:SW_Cherry_MX_1.00u_PCB -> Switch_Keyboard_Hotswap_Kailh:SW_Hotswap_Kailh_MX_1.25u
- SW61: value MENU -> RIGHTCTRL; footprint Button_Switch_Keyboard:SW_Cherry_MX_1.25u_PCB -> Switch_Keyboard_Hotswap_Kailh:SW_Hotswap_Kailh_MX_1.25u
- SW7: value Spacebar -> 6; footprint Button_Switch_Keyboard:SW_Cherry_MX_6.25u_PCB -> Switch_Keyboard_Hotswap_Kailh:SW_Hotswap_Kailh_MX_1.00u
- SW8: value Right_Ctrl -> 7; footprint Button_Switch_Keyboard:SW_Cherry_MX_1.25u_PCB -> Switch_Keyboard_Hotswap_Kailh:SW_Hotswap_Kailh_MX_1.00u
- SW9: value Right_Alt -> 8; footprint Button_Switch_Keyboard:SW_Cherry_MX_1.25u_PCB -> Switch_Keyboard_Hotswap_Kailh:SW_Hotswap_Kailh_MX_1.00u
- moved SW4 257.4 mm to (120.0, 79.0)
- moved SW5 234.2 mm to (139.4, 79.0)
- moved SW6 211.8 mm to (158.9, 79.0)
- moved SW14 209.2 mm to (324.4, 79.0)
- moved SW8 168.2 mm to (197.9, 79.0)
- moved SW28 167.0 mm to (329.4, 98.5)
- moved SW27 161.8 mm to (305.1, 98.5)
- moved SW54 161.1 mm to (64.0, 157.0)
- moved SW55 156.0 mm to (88.5, 157.0)
- moved SW41 154.5 mm to (321.4, 118.0)
- moved C1 151.4 mm to (331.5, 57.0)
- moved SW56 151.0 mm to (113.0, 157.0)
- moved R3 148.4 mm to (324.8, 58.0), turned to 0 degrees
- moved SW40 142.4 mm to (289.9, 118.0)
- moved C6 130.4 mm to (332.5, 63.5), turned to -90 degrees
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Connections:
- D156 pad 2: /COL12 -> /COL13
- SW1 pad 1: Net-(D64-K) -> Net-(D63-K)
- SW1 pad 2: /ROW1 -> /ROW0
- SW10 pad 1: Net-(D67-K) -> Net-(D133-K)
- SW10 pad 2: /ROW4 -> /ROW0
- SW11 pad 1: Net-(D75-K) -> Net-(D140-K)
- SW11 pad 2: /ROW4 -> /ROW0
- SW12 pad 1: Net-(D83-K) -> Net-(D147-K)
- SW12 pad 2: /ROW4 -> /ROW0
- SW13 pad 1: Net-(D158-K) -> Net-(D154-K)
- SW13 pad 2: /ROW4 -> /ROW0
- SW14 pad 1: Net-(D63-K) -> Net-(D161-K)
- SW15 pad 1: Net-(D71-K) -> Net-(D64-K)
- SW15 pad 2: /ROW0 -> /ROW1
- SW16 pad 1: Net-(D79-K) -> Net-(D72-K)
- SW16 pad 2: /ROW0 -> /ROW1
- SW17 pad 1: Net-(D87-K) -> Net-(D80-K)
- SW17 pad 2: /ROW0 -> /ROW1
- SW18 pad 1: Net-(D95-K) -> Net-(D88-K)
- SW18 pad 2: /ROW0 -> /ROW1
- SW19 pad 1: Net-(D103-K) -> Net-(D96-K)
- SW19 pad 2: /ROW0 -> /ROW1
- SW2 pad 1: Net-(D65-K) -> Net-(D71-K)
- SW2 pad 2: /ROW2 -> /ROW0
- SW20 pad 1: Net-(D111-K) -> Net-(D104-K)
- SW20 pad 2: /ROW0 -> /ROW1
- SW21 pad 1: Net-(D119-K) -> Net-(D112-K)
- SW21 pad 2: /ROW0 -> /ROW1
- SW22 pad 1: Net-(D126-K) -> Net-(D120-K)
- SW22 pad 2: /ROW0 -> /ROW1
- SW23 pad 1: Net-(D133-K) -> Net-(D127-K)
- SW23 pad 2: /ROW0 -> /ROW1
- SW24 pad 1: Net-(D140-K) -> Net-(D134-K)
- SW24 pad 2: /ROW0 -> /ROW1
- SW25 pad 1: Net-(D147-K) -> Net-(D141-K)
- SW25 pad 2: /ROW0 -> /ROW1
- SW26 pad 1: Net-(D154-K) -> Net-(D148-K)
- SW26 pad 2: /ROW0 -> /ROW1
- SW27 pad 1: Net-(D72-K) -> Net-(D155-K)
- SW28 pad 1: Net-(D80-K) -> Net-(D162-K)
- SW29 pad 1: Net-(D88-K) -> Net-(D65-K)
- SW29 pad 2: /ROW1 -> /ROW2
- SW3 pad 1: Net-(D66-K) -> Net-(D79-K)
- SW3 pad 2: /ROW3 -> /ROW0
- SW30 pad 1: Net-(D96-K) -> Net-(D73-K)
- SW30 pad 2: /ROW1 -> /ROW2
- SW31 pad 1: Net-(D104-K) -> Net-(D81-K)
- SW31 pad 2: /ROW1 -> /ROW2
- SW32 pad 1: Net-(D112-K) -> Net-(D89-K)
- SW32 pad 2: /ROW1 -> /ROW2
- SW33 pad 1: Net-(D120-K) -> Net-(D97-K)
- SW33 pad 2: /ROW1 -> /ROW2
- SW34 pad 1: Net-(D127-K) -> Net-(D105-K)
- SW34 pad 2: /ROW1 -> /ROW2
- SW35 pad 1: Net-(D134-K) -> Net-(D113-K)
- SW35 pad 2: /ROW1 -> /ROW2
- SW36 pad 1: Net-(D141-K) -> Net-(D121-K)
- SW36 pad 2: /ROW1 -> /ROW2
- SW37 pad 1: Net-(D148-K) -> Net-(D128-K)
- SW37 pad 2: /ROW1 -> /ROW2
- SW38 pad 1: Net-(D155-K) -> Net-(D135-K)
- SW38 pad 2: /ROW1 -> /ROW2
- SW39 pad 1: Net-(D162-K) -> Net-(D142-K)
- SW39 pad 2: /ROW1 -> /ROW2
- SW4 pad 1: Net-(D161-K) -> Net-(D87-K)
- SW40 pad 1: Net-(D73-K) -> Net-(D149-K)
- SW41 pad 1: Net-(D81-K) -> Net-(D156-K)
- SW42 pad 1: Net-(D89-K) -> Net-(D66-K)
- SW42 pad 2: /ROW2 -> /ROW3
- SW43 pad 1: Net-(D97-K) -> Net-(D74-K)
- SW43 pad 2: /ROW2 -> /ROW3
- SW44 pad 1: Net-(D105-K) -> Net-(D82-K)
- SW44 pad 2: /ROW2 -> /ROW3
- SW45 pad 1: Net-(D113-K) -> Net-(D90-K)
- SW45 pad 2: /ROW2 -> /ROW3
- SW46 pad 1: Net-(D121-K) -> Net-(D98-K)
- SW46 pad 2: /ROW2 -> /ROW3
- SW47 pad 1: Net-(D128-K) -> Net-(D106-K)
- SW47 pad 2: /ROW2 -> /ROW3
- SW48 pad 1: Net-(D135-K) -> Net-(D114-K)
- SW48 pad 2: /ROW2 -> /ROW3
- SW49 pad 1: Net-(D142-K) -> Net-(D122-K)
- SW49 pad 2: /ROW2 -> /ROW3
- SW5 pad 1: Net-(D156-K) -> Net-(D95-K)
- SW5 pad 2: /ROW2 -> /ROW0
- SW50 pad 1: Net-(D149-K) -> Net-(D129-K)
- SW50 pad 2: /ROW2 -> /ROW3
- SW51 pad 1: Net-(D74-K) -> Net-(D136-K)
- SW52 pad 1: Net-(D82-K) -> Net-(D143-K)
- SW53 pad 1: Net-(D90-K) -> Net-(D150-K)
- SW54 pad 1: Net-(D98-K) -> Net-(D67-K)
- SW54 pad 2: /ROW3 -> /ROW4
- SW55 pad 1: Net-(D106-K) -> Net-(D75-K)
- SW55 pad 2: /ROW3 -> /ROW4
- SW56 pad 1: Net-(D114-K) -> Net-(D83-K)
- SW56 pad 2: /ROW3 -> /ROW4
- SW57 pad 1: Net-(D122-K) -> Net-(D115-K)
- SW57 pad 2: /ROW3 -> /ROW4
- SW58 pad 1: Net-(D129-K) -> Net-(D144-K)
- SW58 pad 2: /ROW3 -> /ROW4
- SW59 pad 1: Net-(D136-K) -> Net-(D151-K)
- SW59 pad 2: /ROW3 -> /ROW4
- SW6 pad 1: Net-(D150-K) -> Net-(D103-K)
- SW6 pad 2: /ROW3 -> /ROW0
- SW60 pad 1: Net-(D143-K) -> Net-(D158-K)
- SW60 pad 2: /ROW3 -> /ROW4
- SW61 pad 1: Net-(D151-K) -> Net-(D165-K)
- SW7 pad 1: Net-(D115-K) -> Net-(D111-K)
- SW7 pad 2: /ROW4 -> /ROW0
- SW8 pad 1: Net-(D165-K) -> Net-(D119-K)
- SW8 pad 2: /ROW4 -> /ROW0
- SW9 pad 1: Net-(D144-K) -> Net-(D126-K)
- SW9 pad 2: /ROW4 -> /ROW0
Routing:
- net +5V: track 2321.5 -> 365.4 mm, vias 71 -> 12
- net /COL6: track 186.3 -> 496.8 mm, vias 2 -> 3
- net /COL7: track 171.7 -> 477.5 mm, vias 2 -> 3
- net /COL5: track 137.2 -> 428.7 mm, vias 2 -> 3
- net /COL4: track 122.3 -> 411.4 mm, vias 2 -> 3
- net /COL3: track 139.0 -> 385.6 mm, vias 2 -> 3
- net /SCL: track 69.2 -> 268.0 mm, vias 2 -> 1
- net /SDA: track 69.0 -> 267.2 mm, vias 4 -> 1
- net /LED-DAISY: track 116.8 -> 309.6 mm, vias 3 -> 1
- net /D-: track 30.1 -> 216.4 mm, vias 2 -> 6
- net /D+: track 30.0 -> 206.1 mm, vias 2 -> 4
- net /COL2: track 171.3 -> 339.1 mm, vias 0 -> 1
- net /COL1: track 193.4 -> 359.5 mm, vias 0 -> 1
- net /COL12: track 288.1 -> 131.6 mm, vias 2 -> 1
- net /COL13: track 284.6 -> 133.8 mm, vias 2 -> 1
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- added copper zone on B.Cu, net +5V
- added copper zone on F.Cu, net +5V
Other:
- board size 305.9 x 124.4 mm -> 308.5 x 129 mm
- board text removed: "Cooked by - CreatorPoints [Shrestangsu Dutta]"

Commit message: Final push before ship
Parts:
- R1, R2: moved to F.Cu
Routing:
- net Net-(J1-CC2): vias 1 -> 0
- net Net-(J1-CC1): vias 5 -> 4

Commit message: change the pcb-kicad from V2 to V3
Parts:
- R1, R2: moved to B.Cu
- moved R2 189.1 mm to (293.2, 46.3)
- moved J1 187.8 mm to (295.8, 45.3)
- moved R1 187.2 mm to (297.8, 46.3)
- moved U4 173.5 mm to (295.5, 52.5), turned to -90 degrees
- moved U3 132.9 mm to (267.4, 49.0)
- moved C5 23.2 mm to (311.5, 49.0)
- moved C4 17.5 mm to (318.5, 48.0), turned to -90 degrees
- moved C6 15.8 mm to (323.0, 51.0), turned to 0 degrees
- moved C3 12.4 mm to (311.5, 60.5)
- moved C2 3.00 mm to (320.5, 60.5)
- moved R3 1.00 mm to (324.8, 57.0)
Routing:
- net +5V: track 365.4 -> 180.0 mm, vias 12 -> 7
- net /D+: track 206.1 -> 28.0 mm, vias 4 -> 6
- net /D-: track 216.4 -> 44.3 mm
- net /3.3V: track 386.8 -> 345.2 mm, vias 12 -> 10
- net Net-(J1-D--PadA7): track 33.6 -> 5.40 mm
- net Net-(J1-CC1): track 28.4 -> 2.78 mm, vias 4 -> 1
- net Net-(J1-D+-PadA6): track 22.3 -> 5.14 mm
- net GND: track 118.4 -> 129.1 mm, vias 34 -> 32
- net Net-(J1-CC2): track 9.06 -> 2.78 mm, vias 0 -> 1
- net /ROW3: track 438.5 -> 440.3 mm
- net /ROW4: track 450.4 -> 452.1 mm
- net Net-(U1-BOOT0): track 7.94 -> 6.94 mm
Other:
- board size 308.5 x 129 mm -> 308.5 x 130 mm
